File: Crnic_PTP_Project1/Crnic_PTP_Project1.kicad_pcb (KiCad board)
At the start: 2 copper layers, 45 parts, among them U1 LM2574N-5, U2 4027, U3 4027, U4 74LS47, U5 NE555P, U6 SN74LVC1G11, U7 SA39-12EWA

Commit message: Manufacturing
Parts:
- moved R15 1.75 mm to (180.0, 87.5)
- moved R14 0.98 mm to (180.1, 108.5)
- moved R17 0.80 mm to (180.0, 91.0)
- turned R19 to -90 degrees
- turned R20 to -90 degrees
Routing:
- net +5V: track 183.9 -> 239.8 mm, vias 4 -> 10
- net Q3: track 26.2 -> 78.7 mm, vias 8 -> 14
- net Clock: track 6.40 -> 49.0 mm, vias 0 -> 8
- net Q0: track 21.5 -> 58.0 mm
- net Reset: track 0.00 -> 35.6 mm, vias 0 -> 4
- net Net-(U5-DIS): track 15.0 -> 40.8 mm, vias 2 -> 0
- net Q1: track 36.5 -> 58.5 mm, vias 4 -> 10
- net Net-(U4-BI): track 0.00 -> 21.5 mm
- net Net-(U4-e): track 0.00 -> 15.1 mm, vias 0 -> 2
- net GND: track 48.1 -> 59.4 mm, vias 6 -> 10
- net Q2: track 28.6 -> 36.6 mm
- net Net-(U5-THR): track 11.7 -> 19.4 mm
- net Net-(U4-d): track 0.00 -> 6.51 mm
- net Net-(U4-c): track 0.00 -> 6.42 mm
- net Net-(U4-a): track 0.00 -> 6.37 mm
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Other:
- board outline added: 100 x 80 mm
- board text added: "PTP - BCD counter Kristijan Crnić"
